File: NeoXym/XYMPOWER.kicad_sch (KiCad schematic)
At the start: 7 parts, among them U10 74AHCT04, U15 74HCT00, U16 74HCT14, U4 74HCT32, U5 74HCT00, U6 74HCT09, U8 74LS10

Commit message: modified:   NeoXym/CPU_MEM_IOCTRL.kicad_sch 	modified:   NeoXym/XYMGLUE.kicad_sch 	modified:   NeoXym/XYMPOWER.kicad_sch
Parts:
- added C1, C12, C13, C14, C15, C6: 220µF, symbol Device:C_Polarized_Small
- added C10, C11, C7, C8, C9: 10µF, symbol Device:C_Polarized_Small
- added C16, C17, C18, C19, C20, C21, C22: 220nF, symbol Device:C_Small
- added C30, C31: 22pF, symbol Device:C_Small
- added J11: DE9_Receptacle, Connector_Dsub:DSUB-9_Female_EdgeMount_P2.77mm, symbol Connector:DE9_Receptacle
- added J12: DE9_Plug, Connector_Dsub:DSUB-9_Female_EdgeMount_P2.77mm, symbol Connector:DE9_Plug
- added J9: USB_B, symbol Connector:USB_B
- added R16: 100R, Resistor_THT:R_Axial_DIN0207_L6.3mm_D2.5mm_P10.16mm_Horizontal, symbol Device:R_US
- added R17: 100R, symbol Device:R_US
- added U19: MAX232, symbol Interface_UART:MAX232
- added U21: CH340G, Package_SO:SOIC-16_3.9x9.9mm_P1.27mm, symbol Interface_USB:CH340G
- added X2: 12MHz, symbol Device:Crystal
- U10: value 74AHCT04 -> 74HCT04
- U8: value 74LS10 -> 74HCT10
Connections:
- net +5V: now also C11.1, C8.2, U19.16 (VCC)
- net GND: now also C10.1, C11.2, C30.2, C31.2, J11.5, J12.5, J9.4 (GND), J9.5 (Shield), R16.2, R17.2, U19.15 (GND), U21.1 (GND)
- new net: J11.1, R17.1
- new net: J12.1, R16.1
- new net: J12.4, J12.6
- new net: J12.7, J12.8
- new net: C31.1, U21.8 (XO), X2.2
- new net: C10.2, U19.6 (VS-)
- new net: J9.2 (D-), U21.6 (UD-)
- new net: J9.3 (D+), U21.5 (UD+)
- new net: C30.1, U21.7 (XI), X2.1
- new net: C9.1, U19.4 (C2+)
- new net: C9.2, U19.5 (C2-)
- new net: C8.1, U19.2 (VS+)
- new net: J11.4, J11.6
- new net: J11.7, J11.8
- new net: C7.1, U19.1 (C1+)
- new net: C7.2, U19.3 (C1-)
- new net RI_DTE: J12.9
- new net RxD: U19.12 (R1OUT), U21.2 (TXD)
- new net RxDBG: J11.3, U19.13 (R1IN)
- new net RxDT: U19.9 (R2OUT)
- new net RxDTE: J12.2, U19.8 (R2IN)
- new net TxD: U19.11 (T1IN), U21.3 (RXD)
- new net TxDBG: J11.2, U19.14 (T1OUT)
- new net TxDT: U19.10 (T2IN)
- new net TxDTE: J12.3, U19.7 (T2OUT)
- new net VBUS: J9.1 (VBUS)
- no-connect marks 0 -> 7
Other:
- note added: "RS-232 DCE (Debug) Port"
- note added: "RS-232 DTE (Host) Port"
- note added: "USB-VCP Debug Port"

Commit message: modified:   CPU_MEM_IOCTRL.kicad_sch 	modified:   XYMGLUE.kicad_sch 	modified:   XYMPOWER.kicad_sch
Parts:
- added C26: 2.2µF, symbol Device:C_Small
- added C33: 30pF, symbol Device:C_Small
- added C34: 18pF, symbol Device:C_Small
- added R18: 1Meg, symbol Device:R_US
- added U12: W65C51N, Package_DIP:DIP-28_W15.24mm_Socket, symbol 65xx:W65C51N
- added X3: 11.059MHz, symbol Device:Crystal_Small
Connections:
- net +5V: now also C16.1, C17.1, C18.1, C19.1, C20.1, C21.1, C22.1, U10.14 (VCC), U15.14 (VCC), U16.14 (VCC), U4.14 (VCC), U5.7 (GND), U6.14 (VCC), U8.14 (VCC), C26.1, U12.15 (VCC), U12.2 (CS0)
- net GND: now also C16.2, C17.2, C18.2, C19.2, C20.2, C21.2, C22.2, U10.7 (GND), U15.7 (GND), U16.7 (GND), U4.7 (GND), U5.14 (VCC), U6.7 (GND), U8.7 (GND), C26.2, C33.2, C34.2, U12.1 (GND), U12.16 (~{DCD}), U12.17 (~{DSR}), U12.9 (~{CTS})
- net RxDT: now also U12.12 (Rx_Data)
- net TxDT: now also U12.10 (Tx_Data)
- new net: C33.1, R18.1, U12.6 (XTLI), X3.1
- new net: C34.1, R18.2, U12.7 (XLT0), X3.2
- new net ADDR0: U12.13 (RS0)
- new net ADDR1: U12.14 (RS1)
- new net DB0: U12.18 (D0)
- new net DB1: U12.19 (D1)
- new net DB2: U12.20 (D2)
- new net DB3: U12.21 (D3)
- new net DB4: U12.22 (D4)
- new net DB5: U12.23 (D5)
- new net DB6: U12.24 (D6)
- new net DB7: U12.25 (D7)
- new net P2: U12.27 (PHI2)
- new net RW: U12.28 (R/~{W})
- new net ~{ACIA1}: U12.3 (~{CS1})
- new net ~{ACIAIRQ}: U12.26 (~{IRQ})
- new net ~{RST}: U12.4 (~{RESET})
- no-connect marks 7 -> 10
Other:
- note added: "DTE (Host) UART"
- moved on the sheet: C16, C17, C18, C19, C20, C21, C22, U10G, U15E, U4E, U5E
